File: 01_input.kicad_sch (KiCad schematic)
At the start: 27 parts, among them J1 0533980471, U1 VOS618A, U2 LMR51406YDBV

Commit message: Add personal library
Parts:
- L1: footprint Inductor_SMD:L_TDK_VLS3015CX -> Personal_Lib:L_TDK_VLS3015CX
Changed lines of the file:
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@@
 			)
 		)
-		(property "Footprint" "Inductor_SMD:L_TDK_VLS3015CX"
+		(property "Footprint" "Personal_Lib:L_TDK_VLS3015CX"
 			(at 113.03 147.32 0)
 			(effects
