File: 01_input.kicad_sch (KiCad schematic)
At the start: 27 parts, among them J1 0533980471, U1 VOS618A, U2 LMR51406YDBV

Commit message: fix library name
Parts:
- D3: symbol Personal_lib:VESD05B1-02V -> Personal_Lib:VESD05B1-02V
- L1: symbol Personal_lib:L_WindingIndicator -> Personal_Lib:L_WindingIndicator
- U2: symbol Personal_lib:LMR51406YDBV -> Personal_Lib:LMR51406YDBV
Changed lines of the file:
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@@
 	)
 	(symbol
-		(lib_id "Personal_lib:LMR51406YDBV")
+		(lib_id "Personal_Lib:LMR51406YDBV")
 		(at 90.17 142.24 0)
 		(unit 1)
@@
 	)
 	(symbol
-		(lib_id "Personal_lib:L_WindingIndicator")
+		(lib_id "Personal_Lib:L_WindingIndicator")
 		(at 113.03 147.32 90)
 		(unit 1)
@@
 	)
 	(symbol
-		(lib_id "Personal_lib:VESD05B1-02V")
+		(lib_id "Personal_Lib:VESD05B1-02V")
 		(at 118.11 85.09 270)
 		(unit 1)
