File: 02_mcu.kicad_sch (KiCad schematic)
At the start: 31 parts, among them J2 0533980571, U3 MSPM0C1104SDDFR, U4 TLC59208F, U5 VEML7700, U6 TLV803E

Commit message: fix library name
Parts:
- U3: symbol Personal_lib:MSPM0C1104SDDFR -> Personal_Lib:MSPM0C1104SDDFR
- U4: symbol Personal_lib:TLC59208F -> Personal_Lib:TLC59208F
- U5: symbol Personal_lib:VEML7700 -> Personal_Lib:VEML7700
- U6: symbol Personal_lib:TLV803ExxxDBZ -> Personal_Lib:TLV803ExxxDBZ
Changed lines of the file:
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@@
 	)
 	(symbol
-		(lib_id "Personal_lib:VEML7700")
+		(lib_id "Personal_Lib:VEML7700")
 		(at 158.75 151.13 0)
 		(unit 1)
@@
 	)
 	(symbol
-		(lib_id "Personal_lib:MSPM0C1104SDDFR")
+		(lib_id "Personal_Lib:MSPM0C1104SDDFR")
 		(at 54.61 59.69 0)
 		(unit 1)
@@
 	)
 	(symbol
-		(lib_id "Personal_lib:TLV803ExxxDBZ")
+		(lib_id "Personal_Lib:TLV803ExxxDBZ")
 		(at 82.55 154.94 0)
 		(unit 1)
@@
 	)
 	(symbol
-		(lib_id "Personal_lib:TLC59208F")
+		(lib_id "Personal_Lib:TLC59208F")
 		(at 195.58 80.01 0)
 		(unit 1)
